File: Main Board/MoritzKlein-VCA.kicad_sch (KiCad schematic)
At the start: 65 parts, among them J1 Signal In 1, J10 Conn_01x06, J2 Out 1, J3 CV In 1, J4 Signal In 2, J5 Out 2, J6 CV In 2, J7 Conn_01x06, J8 Conn_01x06, J9 Conn_01x06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

Commit message: Upload Schematics
Other:
- note added: "Power"
- title: (none) -> KOSMO - Moritz Klein - VCA
Changed lines of the file:
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@@
 (kicad_sch
-	(version 20231120)
+	(version 20250114)
 	(generator "eeschema")
-	(generator_version "8.0")
+	(generator_version "9.0")
 	(paper "A4")
+	(title_block
+		(title "KOSMO - Moritz Klein - VCA")
+	)
+	(rectangle
+		(start 15.24 160.02)
+		(end 166.37 196.85)
+		(stroke
+			(width 0)
+			(type default)
+		)
+		(fill
+			(type none)
+		)
+	)
+	(text "Power"
+		(exclude_from_sim no)
+		(at 17.78 158.75 0)
+		(effects
+			(font
+				(size 1.27 1.27)
+			)
+		)
+	)
 	(junction
 		(at 64.77 85.09)
@@
 		)
 	)
+	(embedded_fonts no)
 )
